File: CORTICAL EXOSLEEVE.kicad_sch (KiCad schematic)
At the start: 29 parts, among them J1 ESP32-S3 DevKit (Left), J2 Screw_Terminal_01x03, J3 ESP32-S3 DevKit (Right), J4 HYDRAULIC_VALVE, J5 Barrel_Jack_Switch_Pin3Ring, J6 Conn_01x02_Pin, Q1 IRLZ44N, Q2 PN2222A, U2 INA333xxDGK, U3 MP1584EN Buck, U4 MT3608 Boost Module, U5 MCP6001-OT

Commit message: docs: add file-level SPDX headers to firmware, hardware title blocks, and markdown
Other:
- company: (none) -> Prat (pratkan)
- title: (none) -> CORTICAL_EXOSLEEVE - sEMG Hydraulic Controller
Changed lines of the file:
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@@
 	(generator_version "9.0")
 	(paper "A4")
+	(title_block
+		(title "CORTICAL_EXOSLEEVE - sEMG Hydraulic Controller")
+		(date "2026-08-15")
+		(rev "v1.0.0")
+		(company "Prat (pratkan)")
+		(comment 1 "License: CERN-OHL-S-v2 (Strongly Reciprocal)")
+		(comment 2 "SPDX-License-Identifier: CERN-OHL-S-v2")
+		(comment 3 "Copyright (c) 2026 Prat (pratkan)")
+	)
 	(junction
 		(at 60.96 88.9)
